Commit message: 修改tolerance等 尝试使navthroughpoints丝滑

File: src/pb_rmsimulation/src/rm_nav_bringup/urdf/sentry_robot_real.xacro (robot description, xacro)
@@ -17,5 +17,5 @@
     <visual>
       <geometry>
-        <box size="0.2 .3 .1"/>
+        <box size="0.3 0.3 .3"/>
       </geometry>
       <origin rpy="0 0 ${PI/2}" xyz="0 0 0.05"/>
